File: KiCad/MamaMitte_Memory.sch (KiCad schematic (older format))
At the start: 2 parts, among them U1 BANDAI2003, U3 MBM29LV800TA

Commit message: Add footprints and assign nets
Assigned and placed footprints, and assigned nets to vias.
Parts:
- U1: footprint (none) -> MamaMitte:LQFP-48_7x7mm_P0.5mm
- U3: footprint (none) -> MamaMitte:TSOP-I-48_18.4x12mm_P0.5mm
Changed lines of the file:
@@
 $EndDescr
 $Comp
-L power:GND #PWR?
+L power:GND #PWR0128
 U 1 1 609524FD
 P 5875 4050
-F 0 "#PWR?" H 5875 3800 50  0001 C CNN
+F 0 "#PWR0128" H 5875 3800 50  0001 C CNN
 F 1 "GND" H 5880 3877 50  0000 C CNN
 F 2 "" H 5875 4050 50  0001 C CNN
@@
 	6250 4050 5875 4050
 $Comp
-L power:+3.3V #PWR?
+L power:+3.3V #PWR0129
 U 1 1 609E3FD1
 P 2700 3850
-F 0 "#PWR?" H 2700 3700 50  0001 C CNN
+F 0 "#PWR0129" H 2700 3700 50  0001 C CNN
 F 1 "+3.3V" H 2715 4023 50  0000 C CNN
 F 2 "" H 2700 3850 50  0001 C CNN
@@
 	3200 3850 2700 3850
 $Comp
-L power:+3.3V #PWR?
+L power:+3.3V #PWR0130
 U 1 1 60A26E4E
 P 8050 4350
-F 0 "#PWR?" H 8050 4200 50  0001 C CNN
+F 0 "#PWR0130" H 8050 4200 50  0001 C CNN
 F 1 "+3.3V" H 8065 4523 50  0000 C CNN
 F 2 "" H 8050 4350 50  0001 C CNN
@@
 	7700 4350 8050 4350
 $Comp
-L power:+3.3V #PWR?
+L power:+3.3V #PWR0131
 U 1 1 60A06B5F
 P 4925 3650
-F 0 "#PWR?" H 4925 3500 50  0001 C CNN
+F 0 "#PWR0131" H 4925 3500 50  0001 C CNN
 F 1 "+3.3V" H 4940 3823 50  0000 C CNN
 F 2 "" H 4925 3650 50  0001 C CNN
@@
 	6250 2550 6250 2650
 $Comp
-L power:GND #PWR?
+L power:GND #PWR0132
 U 1 1 6096C97D
 P 5875 2550
-F 0 "#PWR?" H 5875 2300 50  0001 C CNN
+F 0 "#PWR0132" H 5875 2300 50  0001 C CNN
 F 1 "GND" H 5880 2377 50  0000 C CNN
 F 2 "" H 5875 2550 50  0001 C CNN
@@
 	6250 2550 5875 2550
 $Comp
-L power:GND #PWR?
+L power:GND #PWR0133
 U 1 1 6096A048
 P 5875 3050
-F 0 "#PWR?" H 5875 2800 50  0001 C CNN
+F 0 "#PWR0133" H 5875 2800 50  0001 C CNN
 F 1 "GND" H 5880 2877 50  0000 C CNN
 F 2 "" H 5875 3050 50  0001 C CNN
@@
 CE
 $Comp
-L power:GND #PWR?
+L power:GND #PWR0134
 U 1 1 60929D20
 P 4925 4650
-F 0 "#PWR?" H 4925 4400 50  0001 C CNN
+F 0 "#PWR0134" H 4925 4400 50  0001 C CNN
 F 1 "GND" H 4930 4477 50  0000 C CNN
 F 2 "" H 4925 4650 50  0001 C CNN
@@
 	4600 4650 4925 4650
 $Comp
-L power:GND #PWR?
+L power:GND #PWR0135
 U 1 1 60922A17
 P 4925 2750
-F 0 "#PWR?" H 4925 2500 50  0001 C CNN
+F 0 "#PWR0135" H 4925 2500 50  0001 C CNN
 F 1 "GND" H 4930 2577 50  0000 C CNN
 F 2 "" H 4925 2750 50  0001 C CNN
@@
 F 0 "U1" H 6975 5175 60  0000 C CNN
 F 1 "BANDAI2003" H 6975 5075 60  0000 C CNN
-F 2 "" H 6950 3650 60  0001 C CNN
+F 2 "MamaMitte:LQFP-48_7x7mm_P0.5mm" H 6950 3650 60  0001 C CNN
 F 3 "" H 6950 3650 60  0001 C CNN
 	1    6950 3700
@@
 F 0 "U3" H 3900 5187 60  0000 C CNN
 F 1 "MBM29LV800TA" H 3900 5081 60  0000 C CNN
-F 2 "" H 3900 3700 60  0001 C CNN
+F 2 "MamaMitte:TSOP-I-48_18.4x12mm_P0.5mm" H 3900 3700 60  0001 C CNN
 F 3 "" H 3900 3700 60  0001 C CNN
 	1    3900 3700

Commit message: Update schematic
Fix Bandai 2003 pinout and RTC power.
Connections:
- net A15: no longer U1.15 (SA15), U3.1 (A15)
- net A16: no longer U1.14 (SA16), U3.48 (A16)
- net A17: no longer U1.20 (SA17), U3.17 (A17)
- net A18: no longer U1.19 (SA18), U3.16 (A18)
- net A19 renamed SA19
- net SA19: now also U1.17 (SA19); no longer U1.18 (SA20)
- net A20 renamed SA20
- net SA20: now also U1.18 (SA20); no longer U1.17 (SA19)
- net A21 renamed SA21
- new net SA15: U1.15 (SA15), U3.1 (A15)
- new net SA16: U1.14 (SA16), U3.48 (A16)
- new net SA17: U1.20 (SA17), U3.17 (A17)
- new net SA18: U1.19 (SA18), U3.16 (A18)
Changed lines of the file:
@@
 	6050 3750 6250 3750
 Text Label 6050 3750 0    50   ~ 0
-A21
+SA21
 Wire Wire Line
 	6050 4150 6250 4150
 Text Label 6050 4150 0    50   ~ 0
-A20
+SA19
 Wire Wire Line
 	6050 4250 6250 4250
 Text Label 6050 4250 0    50   ~ 0
-A19
+SA20
 Wire Wire Line
-	2875 3750 3200 3750
-Text Label 2875 3750 0    50   ~ 0
-A21
+	2825 3750 3200 3750
+Text Label 2825 3750 0    50   ~ 0
+SA21
 Wire Wire Line
-	2875 3450 3200 3450
-Text Label 2875 3450 0    50   ~ 0
-A20
+	2825 3450 3200 3450
+Text Label 2825 3450 0    50   ~ 0
+SA20
 Wire Wire Line
-	2875 3350 3200 3350
-Text Label 2875 3350 0    50   ~ 0
-A19
+	2825 3350 3200 3350
+Text Label 2825 3350 0    50   ~ 0
+SA19
 Wire Wire Line
-	2875 4050 3200 4050
-Text Label 2875 4050 0    50   ~ 0
-A18
+	2825 4050 3200 4050
+Text Label 2825 4050 0    50   ~ 0
+SA18
 Wire Wire Line
-	2875 4150 3200 4150
-Text Label 2875 4150 0    50   ~ 0
-A17
+	2825 4150 3200 4150
+Text Label 2825 4150 0    50   ~ 0
+SA17
 Text GLabel 4600 4850 2    50   Input ~ 0
 A0
@@
 	6050 4350 6250 4350
 Text Label 6050 4350 0    50   ~ 0
-A18
+SA18
 Wire Wire Line
 	6050 4450 6250 4450
 Text Label 6050 4450 0    50   ~ 0
-A17
+SA17
 Wire Wire Line
 	6050 3850 6250 3850
 Text Label 6050 3850 0    50   ~ 0
-A16
+SA16
 Wire Wire Line
-	2875 2550 3200 2550
-Text Label 2875 2550 0    50   ~ 0
-A15
+	2825 2550 3200 2550
+Text Label 2825 2550 0    50   ~ 0
+SA15
 Wire Wire Line
 	6050 3950 6250 3950
 Text Label 6050 3950 0    50   ~ 0
-A15
+SA15
 Wire Wire Line
 	4800 2550 4600 2550
 Text Label 4800 2550 2    50   ~ 0
-A16
+SA16
 Wire Wire Line
 	4600 4750 4800 4750
